File: hardware/sensor-hub-carrier/sensor-hub-carrier.kicad_sch (KiCad schematic)
At the start: 6 parts, among them U1 ESP32-S3-DEVKITC-1-N8R2

Commit message: docs: Release Hardware v1.1 (Relay Driver + Expansion Ports)
Parts:
- added D2: 1N4007, Diode_THT:D_DO-41_SOD81_P10.16mm_Horizontal, symbol Diode:1N4007
- added J_EXP1: EXP, Connector_PinSocket_2.54mm:PinSocket_1x08_P2.54mm_Vertical, symbol Connector:Conn_01x08_Socket
- added J_MIC1: INMP441, Connector_PinSocket_2.54mm:PinSocket_1x06_P2.54mm_Vertical, symbol Connector:Conn_01x06_Socket
- added J_RELAY1: 5V, TerminalBlock:TerminalBlock_bornier-2_P5.08mm, symbol Connector:Screw_Terminal_01x02
- added Q1: 2N3904, Package_TO_SOT_THT:TO-92_Inline, symbol Transistor_BJT:2N3904
- added R2: 1K, Resistor_THT:R_Axial_DIN0207_L6.3mm_D2.5mm_P10.16mm_Horizontal, symbol Device:R
- J_POWER1: value Screw_Terminal_01x02 -> +5V
Connections:
- net 3V3: now also J_EXP1.2 (Pin_2), J_MIC1.1 (Pin_1)
- net GND: now also J_EXP1.3 (Pin_3), J_EXP1.4 (Pin_4), J_MIC1.2 (Pin_2), J_MIC1.3 (Pin_3), Q1.1 (E)
- net VCC: now also D2.1 (K), J_EXP1.1 (Pin_1), J_RELAY1.2 (Pin_2)
- net SD: now reaches U1.J1_12 (GPIO8)
- net SD: now also J_MIC1.6 (Pin_6)
- net WS: now reaches U1.J1_15 (GPIO9)
- net WS: now also J_MIC1.5 (Pin_5)
- net SCK: now reaches U1.J1_16 (GPIO10)
- net SCK: now also J_MIC1.4 (Pin_4)
- net GPIO11: now reaches U1.J1_17 (GPIO11)
- net GPIO11: now also R2.2
- net GPIO4: now reaches U1.J1_4 (GPIO4)
- net GPIO4: now also J_EXP1.5 (Pin_5)
- net GPIO5: now reaches U1.J1_5 (GPIO5)
- net GPIO5: now also J_EXP1.6 (Pin_6)
- net GPIO6: now reaches U1.J1_6 (GPIO6)
- net GPIO6: now also J_EXP1.7 (Pin_7)
- net GPIO7: now reaches U1.J1_7 (GPIO7)
- net GPIO7: now also J_EXP1.8 (Pin_8)
- new net: Q1.2 (B), R2.1
- new net: D2.2 (A), J_RELAY1.1 (Pin_1), Q1.3 (C)
- no-connect marks 40 -> 32
Other:
- company: (none) -> Ing Jhon Alexander Hernandez
- title: (none) -> Sensor Hub Carrier
